File: Electronics/usb_uart_dongle_V1.0.0.kicad_sch (KiCad schematic)
At the start: 22 parts, among them IC1 CP2102-GM, J1 61200621721, SW1 SS-3390S-L1

Commit message: V1.0.0
Parts:
- removed JP1, JP2: SolderJumper_3_Open, f:SolderJumper-3_P1.3mm_Open_RoundedPad1.0x1.5mm, symbol Jumper:SolderJumper_3_Open
- added JP3: SolderJumper_2_Open, f:SolderJumper-2_P1.3mm_Open_Pad1.0x1.5mm, symbol Jumper:SolderJumper_2_Open
Connections:
- net +3V3: now also JP3.1 (A); no longer SW1.2
- net RXD: now also SW1.2
- net TXD: now also SW1.5
- net UART_PIN_1: now also SW1.1, SW1.6
- net UART_PIN_2: now also SW1.3, SW1.4
- net at J1.5: now also JP3.2 (B); no longer SW1.1
- no-connect marks 9 -> 8
Other:
- moved on the sheet: D4, J1, R1
